File: Carte_moteur.kicad_pcb (KiCad board)
At the start: 2 copper layers, 113 parts, among them J101 Conn_01x02_Socket, J102 Conn_01x02, J103 Conn_01x02, J104 Conn_01x07, J105 Conn_01x02_Socket, J106 Conn_01x07, J201 Conn_01x05_Pin, J202 Conn_01x04_Pin, J301 Conn_01x05_Pin, J302 Conn_01x04_Pin, J401 Conn_01x05_Pin, J402 Conn_01x04_Pin, J601 Conn_01x06_Pin, J602 USB_B_Mini, Q601 MMBTA44, U101 LD1117S33TR_SOT223, U201 TMC2209, U301 TMC2209, U401 TMC2209, U501 STM32G474RETx, U601 ECMF02-2AMX6, U602 LD1117S33TR_SOT223, U603 STM32F103CBTx, Y601 Crystal_GND24

Commit message: almost done
Parts:
- C503, C504, C505, C506, C508, R510, R511: moved to B.Cu
- moved R518 70.8 mm to (96.0, 99.1), turned to 90 degrees
- moved R519 70.0 mm to (98.3, 99.1), turned to -90 degrees
- moved C505 37.2 mm to (110.2, 110.0), turned to 180 degrees
- moved C504 30.9 mm to (106.2, 109.0)
- moved C506 30.3 mm to (105.2, 102.9), turned to 0 degrees
- moved R511 27.2 mm to (104.1, 109.0), turned to -90 degrees
- moved C508 24.6 mm to (105.2, 106.4), turned to 180 degrees
- moved R510 19.2 mm to (110.5, 102.9)
- moved C503 16.8 mm to (110.5, 104.6)
- moved U101 15.4 mm to (81.5, 114.8)
- moved C103 15.4 mm to (79.2, 107.2)
- moved C105 15.4 mm to (82.3, 107.2)
- moved R516 10.4 mm to (117.1, 102.6), turned to 180 degrees
- moved R513 10.0 mm to (117.1, 105.9), turned to 180 degrees
- moved R517 9.89 mm to (117.1, 104.1), turned to 180 degrees
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Connections:
- J104 pad 4: /micro/T_SWCLK -> /micro/T_SWDIO
- J104 pad 5: /micro/T_SWDIO -> /micro/T_SWCLK
- J104 pad 6: /micro/T_SWO -> /micro/T_JDTI
- J104 pad 7: /micro/T_JDTI -> /micro/T_SWO
- J106 pad 2: /micro/UART4_RX -> /micro/LPUART1_RX
- J106 pad 3: /micro/UART4_TX -> /micro/LPUART1_TX
- J201 pad 2: /micro/TIM1_CH1 -> /micro/TIM5_CH1
- J201 pad 3: /micro/TIM1_CH2 -> /micro/TIM5_CH2
- J201 pad 4: /micro/TIM1_ETR -> /micro/TIM5_ETR
- J301 pad 2: /micro/TIM5_CH1 -> /micro/TIM1_CH1
- J301 pad 3: /micro/TIM5_CH2 -> /micro/TIM1_CH2
- J301 pad 4: /micro/TIM5_ETR -> /micro/TIM1_ETR
- R210 pad 1: /micro/TIM1_CH1 -> /micro/TIM5_CH1
- R211 pad 1: /micro/TIM1_CH2 -> /micro/TIM5_CH2
- R212 pad 1: /micro/TIM1_ETR -> /micro/TIM5_ETR
- R512 pad 1: /micro/TMC1 -> /micro/TMC2
- R513 pad 1: /micro/TMC1 -> /micro/TMC2
- R514 pad 1: /micro/TMC2 -> /micro/TMC1
- R515 pad 1: /micro/TMC2 -> /micro/TMC1
- R523 pad 1: /micro/TIM5_CH1 -> /micro/TIM1_CH1
- R524 pad 1: /micro/TIM5_CH2 -> /micro/TIM1_CH2
- R525 pad 1: /micro/TIM5_ETR -> /micro/TIM1_ETR
- U201 pad 7: /micro/HRTIM_CHA1 -> /micro/HRTIM_CHE1
- U201 pad 8: /micro/HRTIM_CHA2 -> /micro/HRTIM_CHE2
- U301 pad 7: /micro/HRTIM_CHE1 -> /micro/HRTIM_CHA1
- U301 pad 8: /micro/HRTIM_CHE2 -> /micro/HRTIM_CHA2
- U603 pad 12: /micro/LPUART1_RX -> /micro/UART4_RX
- U603 pad 13: /micro/LPUART1_TX -> /micro/UART4_TX
Routing:
- net GND: track 175.8 -> 274.6 mm, vias 14 -> 19
- net +3V3: track 75.2 -> 134.5 mm, vias 0 -> 4
- net +5V: track 0.00 -> 52.9 mm
- net /tmc_motor2/B02: track 68.0 -> 22.4 mm
- net /tmc_motor2/B01: track 60.4 -> 20.1 mm
- net /tmc_motor2/A02: track 49.7 -> 16.4 mm
- net /tmc_motor2/A01: track 49.7 -> 16.6 mm
- net /micro/T_RST: track 2.64 -> 31.8 mm, vias 0 -> 2
- net /micro/SPI1_MOSI: track 0.00 -> 23.4 mm
- net /micro/TMC2: track 56.8 -> 80.2 mm
- net /micro/T_SWO: track 2.54 -> 25.2 mm, vias 0 -> 2
- net /micro/SPI1_MISO: track 0.00 -> 21.7 mm
- net /micro/HRTIM_CHA1: track 17.1 -> 38.0 mm, vias 1 -> 0
- net /micro/TIM5_CH2: track 58.6 -> 38.7 mm, vias 4 -> 1
- net /micro/SPI1_SCK: track 0.00 -> 19.8 mm
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
Commit message: tracks done
Parts:
- removed C501, C507: C, Capacitor_SMD:C_0603_1608Metric_Pad1.08x0.95mm_HandSolder
- moved C104 40.3 mm to (87.6, 157.2)
- moved C102 20.9 mm to (87.6, 148.0)
- moved C101 16.8 mm to (87.6, 134.9)
- moved D601 15.8 mm to (138.5, 112.0)
- moved C601 4.09 mm to (134.2, 111.9)
- moved D602 2.33 mm to (137.0, 108.5)
- moved R101 1.92 mm to (119.9, 112.8)
- moved U602 1.22 mm to (136.5, 116.8)
- moved C604 1.22 mm to (131.4, 104.2)
- moved C606 1.22 mm to (131.4, 105.8)
- moved J602 1.22 mm to (142.6, 104.1)
- moved R603 1.22 mm to (136.2, 102.5)
- moved R604 1.22 mm to (136.2, 104.1)
- moved R605 1.22 mm to (133.7, 100.8)
- moved R606 1.22 mm to (133.7, 99.0)
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Routing:
- net GND: track 274.6 -> 561.1 mm, vias 19 -> 21
- net +BATT: track 7.46 -> 91.1 mm
- net +3V3: track 134.5 -> 205.8 mm, vias 4 -> 7
- net +5V: track 52.9 -> 121.4 mm, vias 0 -> 1
- net /micro/LPUART1_TX: track 0.00 -> 16.0 mm, vias 0 -> 1
- net Net-(D601-K): track 6.16 -> 11.7 mm
- net /stlink/T_NRST: track 13.4 -> 10.3 mm
- net /micro/HRTIM_CHA1: track 38.0 -> 35.3 mm
- net /micro/TIM3_ETR: track 45.0 -> 42.4 mm, vias 0 -> 2
- net /micro/TIM3_CH1: track 39.8 -> 42.3 mm
- net /micro/T_RST: track 31.8 -> 34.2 mm
- net /micro/SPI1_MOSI: track 23.4 -> 21.5 mm
- net /micro/SPI1_SCK: track 19.8 -> 18.1 mm
- net /micro/SPI1_MISO: track 21.7 -> 20.0 mm
- net /micro/LPUART1_RX: track 14.8 -> 13.2 mm
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